Commit message: isaacsim: clamp xArm7 joint2/joint6 URDF limits to the official datasheet
URDF had joint2 at +-2.18 rad (official -2.059..2.0944) and joint6 lower
at -1.75 (official -1.69297). The policy's action clamp uses live joint
limits, so training against the wider range teaches poses the real arm
rejects. XHand hand-joint limits were verified to match the real SDK
(WRS xhand_right model) exactly — no change needed there.

Co-Authored-By: Claude Fable 5 <noreply@anthropic.com>

File: assets/urdf/xarm7_xhand/xarm7_xhand.urdf (robot description, URDF)
Before this commit: robot xarm7_xhand, 22 links, 21 joints
Joints:
- joint joint2: limit lower=-2.18 upper=2.18 effort=50.0 velocity=3.14 -> lower=-2.059 upper=2.0944 effort=50.0 velocity=3.14
- joint joint6: limit lower=-1.75 upper=3.14159265 effort=20.0 velocity=3.14 -> lower=-1.69297 upper=3.14159265 effort=20.0 velocity=3.14

Commit message: isaacsim: fix XHand contact physics — convex decomposition, real inertia, armature
Root cause of the policy wedging objects in the finger gaps instead of
pinching with the fingertips: the XHand reuses its detailed visual mesh as
its collision mesh, and the URDF converter approximated each link with a
single convex hull. Measured inflation is 1.53-3.45x (distal links 2.06x,
thumb base 3.45x) — the hull fills each finger's concave inner face and
bridges the inter-segment gaps, so the object rests on an invisible bulge
belonging to low-friction proximal links. The legacy Sharpa hand shipped
purpose-built convex collision proxies (1.00-1.27x), so a plain hull was
correct there. Friction values/assignment were verified correct and are
unchanged (1.5 on the five distal links, 0.5 elsewhere, per PhysX runtime).

- collider_type=convex_decomposition for the robot (21 -> 336 shapes)
- inertia for all 21 links computed from the true (non-hull) meshes at a
  uniform 1700 kg/m^3: arm 13.80 kg, hand 0.607 kg, matching the quoted
  unit masses. Previously the arm carried flat 1.0 kg placeholders with
  isotropic 0.01 tensors and the hand had no <inertial> at all, so PhysX
  derived finger mass/COM from the *inflated* hulls.
- armature on every joint. Sharpa's 4.2e-4..3.2e-3 dominated its ~1e-6
  link inertias and kept each joint at omega ~40-107 rad/s, zeta ~0.9;
  XHand had none, leaving omega up to 1225 rad/s (omega*dt = 10 at 120 Hz)
  and zeta up to 20. Arm armature levels I_eff to ~0.12 at every joint.
- arm damping 80 -> 11.1: a flat 80 gave zeta 5.9 at the shoulder and 84
  at the wrist (iiwa reference: 0.55-0.89), i.e. a wrist that barely
  responded — plausibly why orientation alignment learned so slowly.
- fingertip pad / palm-center observation offsets measured from geometry,
  replacing placeholders; fingertip body ids now resolved with
  preserve_order because the thumb's pad offset points along a different
  axis and articulation order is not FINGERTIP_LINK_NAMES order.

Co-Authored-By: Claude Fable 5 <noreply@anthropic.com>

File: assets/urdf/xarm7_xhand/xarm7_xhand.urdf (robot description, URDF)
Before this commit: robot xarm7_xhand, 22 links, 21 joints
Links:
- link index_bend_link: mass None -> 0.0235446
- link index_rota_link1: mass None -> 0.0238768
- link index_rota_link2: mass None -> 0.0112549
- link link1: mass 1.0 -> 2.24548
- link link2: mass 1.0 -> 2.69339
- link link3: mass 1.0 -> 1.92619
- link link4: mass 1.0 -> 2.23109
- link link5: mass 1.0 -> 1.33579
- link link6: mass 1.0 -> 1.22414
- link link7: mass 1.0 -> 0.172658
- link link_base: mass 1.0 -> 1.97098
- link mid_link1: mass None -> 0.0238768
- link mid_link2: mass None -> 0.0112549
- link palm: mass None -> 0.332857
- link pinky_link1: mass None -> 0.0238768
- link pinky_link2: mass None -> 0.0112549
- link ring_link1: mass None -> 0.0238768
- link ring_link2: mass None -> 0.0112549
- link thumb_bend_link: mass None -> 0.00595385
- link thumb_rota_link1: mass None -> 0.0576565
- link thumb_rota_link2: mass None -> 0.0462109

Commit message: isaacsim: apply the XHand1 product-manual specs (model 2R32)
Found the official manual (X-Hand 1 Product Manual V1.0, 2024/10) — model
2R32 is exactly the hand in assets/urdf/xhand2R32. It corrects three things
that were previously estimated or simply wrong:

- Joint limits: thumb_joint0 0..1.83 -> 0..1.57, thumb_joint2 -0.175..1.83
  -> 0..1.57, index_joint0 +-0.175 -> -0.087..0.297 (the real index abducts
  17 deg outward but only 5 deg inward; ours was symmetric). The action
  pipeline denormalizes [-1,1] onto these limits, so the policy had been
  learning thumb and abduction poses the hardware cannot reach. The other
  nine joints already matched. Note this also supersedes the WRS library
  values these were first checked against — it carried the same wrong ones.
- Hand mass: official 1.1 kg. A uniform 1700 kg/m^3 (calibrated on the arm,
  which lands at 13.80 kg vs xArm7's quoted ~13.7) gives the hand only
  0.607 kg, so the hand now uses its own 3082 kg/m^3 — a hand is mostly
  motors and gearing, an arm is mostly hollow structure.
- Effort limits: flat 10 Nm -> per-joint 1.9/4.6/5.5-6.1 Nm, from the
  manual's 50 N single-finger max load times each joint's measured lever
  arm to the fingertip pad.

Also records a caveat on the armature values: the manual describes a
Quasi-Direct Drive transmission, whose low reduction reflects far less
rotor inertia than the harmonic-drive-like values borrowed from Sharpa.

Co-Authored-By: Claude Fable 5 <noreply@anthropic.com>

File: assets/urdf/xarm7_xhand/xarm7_xhand.urdf (robot description, URDF)
Before this commit: robot xarm7_xhand, 22 links, 21 joints
Links:
- link index_bend_link: mass 0.0235446 -> 0.0426848
- link index_rota_link1: mass 0.0238768 -> 0.0432872
- link index_rota_link2: mass 0.0112549 -> 0.0204045
- link mid_link1: mass 0.0238768 -> 0.0432872
- link mid_link2: mass 0.0112549 -> 0.0204045
- link palm: mass 0.332857 -> 0.603449
- link pinky_link1: mass 0.0238768 -> 0.0432872
- link pinky_link2: mass 0.0112549 -> 0.0204045
- link ring_link1: mass 0.0238768 -> 0.0432872
- link ring_link2: mass 0.0112549 -> 0.0204045
- link thumb_bend_link: mass 0.00595385 -> 0.010794
- link thumb_rota_link1: mass 0.0576565 -> 0.104528
- link thumb_rota_link2: mass 0.0462109 -> 0.0837775
Joints:
- joint index_joint0: limit lower=-0.175 upper=0.175 effort=10 velocity=3.14 -> lower=-0.087 upper=0.297 effort=5.5 velocity=3.14
- joint index_joint1: limit lower=0.0 upper=1.92 effort=10 velocity=3.14 -> lower=0 upper=1.92 effort=4.6 velocity=3.14
- joint index_joint2: limit lower=0.0 upper=1.92 effort=10 velocity=3.14 -> lower=0 upper=1.92 effort=1.9 velocity=3.14
- joint middle_joint0: limit lower=0.0 upper=1.92 effort=10 velocity=3.14 -> lower=0 upper=1.92 effort=4.6 velocity=3.14
- joint middle_joint1: limit lower=0.0 upper=1.92 effort=10 velocity=3.14 -> lower=0 upper=1.92 effort=1.9 velocity=3.14
- joint pinky_joint0: limit lower=0.0 upper=1.92 effort=10 velocity=3.14 -> lower=0 upper=1.92 effort=4.6 velocity=3.14
- joint pinky_joint1: limit lower=0.0 upper=1.92 effort=10 velocity=3.14 -> lower=0 upper=1.92 effort=1.9 velocity=3.14
- joint ring_joint0: limit lower=0.0 upper=1.92 effort=10 velocity=3.14 -> lower=0 upper=1.92 effort=4.6 velocity=3.14
- joint ring_joint1: limit lower=0.0 upper=1.92 effort=10 velocity=3.14 -> lower=0 upper=1.92 effort=1.9 velocity=3.14
- joint thumb_joint0: limit lower=0.0 upper=1.83 effort=10 velocity=3.14 -> lower=0 upper=1.57 effort=6.1 velocity=3.14
- joint thumb_joint1: limit lower=-1.05 upper=1.57 effort=10 velocity=3.14 -> lower=-1.05 upper=1.57 effort=4.6 velocity=3.14
- joint thumb_joint2: limit lower=-0.175 upper=1.83 effort=10 velocity=3.14 -> lower=0 upper=1.57 effort=1.9 velocity=3.14
