Commit message: isaacsim: roll the hand back to the original 15 deg — the 180 flip hid the thumb
The policy grasps with the four fingers curling on their own: the thumb sits
16 cm from the object and barely flexes (0.78 rad against the index's 3.27),
and the object is not against the palm either. Freezing everything else and
sweeping the thumb through its range shows it could halve that distance — so
it can reach, it just never does.

Cause: this port mounted the hand at the iiwa's 15 deg PLUS 180. That was
chosen to make the fingertip centroid line up with the XHand build's (y=0.074
against 0.086) — a cosmetic match — and it silently put the thumb on the
wrong side. Measured at the home pose:

                    thumb vs fingers (z)   thumb-object minus fingers-object
  original KUKA            -0.005 m                    +2.3 cm
  this port at 195 deg     +0.100 m                   +11.4 cm
  restored to 15 deg       -0.083 m                    -3.3 cm

At 195 deg the thumb rides 10 cm above the fingers and 11 cm further from the
object; at 15 deg it sits just below them and closer than they are, which is
what the original looks like.

This answers why the problem exists at all when the original guides nothing
by reward: the original does not need to. Its mounting puts the thumb in an
opposable position by construction, so closing the fingers yields a
thumb-opposed pinch for free. The reward — verified opposition-agnostic in
both the original and this port — has no term that would recover it once the
geometry stops offering it.

Co-Authored-By: Claude Fable 5 <noreply@anthropic.com>

File: assets/urdf/xarm7_sharpa/xarm7_sharpa.urdf (robot description, URDF)
Before this commit: robot xarm7_sharpa, 43 links, 42 joints
Joints:
- joint sharpa_mount: origin xyz=0 0 0 rpy=0 0 3.403392 -> xyz=0 0 0 rpy=0 0 0.261799
